File: PCB v2.kicad_pcb (KiCad board)
At the start: 4 copper layers, 55 x 49.6 mm, 91 parts, among them J1 Conn_01x02_Pin, J3 6871XX182122_687110182122, J5 Conn_01x03_Pin, J7 Conn_01x07_Pin, U1 LT3483AxS6, U11 OPA4350EA_250, U12 OPA4350EA_250, U13 OPA4350EA_250, U2 LT1761-2.5, U3 LT1964-BYP, U5 AD7606, U6 OPA4350EA_250

Commit message: Eseguite modifiche
Parts:
- moved J5 44.9 mm to (153.3, 80.7), turned to -90 degrees
- moved H3 7.13 mm to (124.8, 116.0)
- moved H4 7.13 mm to (174.7, 116.0)
Routing:
- net +2V5: track 89.7 -> 33.1 mm, vias 9 -> 8
- net S8: track 10.1 -> 39.4 mm, vias 0 -> 2
- net S_sac: track 19.6 -> 40.7 mm, vias 0 -> 2
- net V_sac: track 81.2 -> 69.9 mm, vias 4 -> 6
- net GND: track 191.4 -> 186.3 mm
- net +5V: track 90.0 -> 92.1 mm, vias 2 -> 4
- added copper zone on In2.Cu, net +2V5
- removed copper zone on F.Cu, net +2V5
Other:
- board size 55 x 49.6 mm -> 55 x 42.7 mm
- board text added: "+2V5"
- board text added: "+5V"
- board text added: "-2V5"
- board text added: "-5V"
- board text added: "BUSY"
- board text added: "CONVST"
- board text added: "GND"
- board text added: "RESET"
- board text added: "S8"
- board text added: "SPI_CS"
- board text added: "SPI_MISO"
- board text added: "SPI_SCK"
- board text added: "S_SAC"
- board text added: "Vdrive"
