File: PCB/FOGLIO2.kicad_sch (KiCad schematic)
At the start: 56 parts, among them U11 OPA4350EA_250, U12 OPA4350EA_250, U13 OPA4350EA_250, U6 OPA4350EA_250

Commit message: Modifiche accordate fatte
Connections:
- net in-_b3: now also R50.2; no longer R50.1
- net out_a3: now also R50.1; no longer R50.2
- net vout1 renamed Vout1
- net vout2 renamed Vout2
- net vout5 renamed Vout5
- net vout6 renamed Vout6
- net vout7 renamed Vout7
Other:
- moved on the sheet: R50
