File: PCB/PCB v2.kicad_sch (KiCad schematic)
At the start: 0 parts

Commit message: Swap AD7606 for ADS131M08, rework analog front-end and USB input
Schematic-only changes; the PCB has not been updated from the schematic
yet. PCB/CHANGELOG-2026-09-28-ADC-swap.md has the per-part details: every
added/removed part with its pin-to-net list, the netlist diff (before ->
after) and the ERC counts.

1. ADC swap (FOGLIO1)
- Remove the AD7606 (U5) and parts that only served it: C29-C32, C45-C47,
  BUSY LED D3/R8 and the old 1x07 J7.
- Wire up the ADS131M08 (U2): internal 1.2 V reference with 100n on REFIN,
  XTAL2 no-connect, AINxN tied to GND.
- Per-channel divider + anti-alias RC (R61-R76 1.1k/1k, C48-C55 10n C0G):
  op-amp swing +-2.45 V -> +-1.17 V for the +-1.2 V ADC full scale,
  fc ~30 kHz. Channel 7 now digitises the sacrificial-sensor output Vsac.
- ADC supply: U7 TPS7A2033 LDO from +5V -> +3.3VA (AVDD), FB1 -> +3V3
  (DVDD, U3, pull-ups). 1.7 V headroom gives full PSRR, which a passive
  filter on raw VBUS could not.
- Clock from the STM32H7 (MCO2, 5.12 MHz, OSR 256 -> 10 kSPS):
  MCU_CLK -> U3 74LVC1G17 Schmitt buffer -> R80 33R -> CLKIN, with R79
  100k pull-down so CLKIN never floats.
- SPI: R81/R82 33R source terminations on DOUT/DRDY, R77/R78 10k pull-ups
  on CS and SYNC/RESET.
- New 2x06 J7 with GND next to CLK and SCLK.
- Vsac brought from the SENSORS sheet through a new sheet pin (plain wire
  on the root sheet).
- FOGLIO1 paper A4 -> A3. PWR_FLAG added on GND (pre-existing ERC error).

2. Op-amp section swap (FOGLIO2)
- U6 and U13, the two quads next to J3, now hold all 8 first stages
  (S1-S7 and S_sac); U11/U12 hold the 7 difference amps. The
  high-impedance sensor traces can now stay short and on F.Cu.
- Section order chosen from the J3/op-amp pad positions so the sensor
  traces can be routed without crossings.
- Spare section U12-D wired as a follower with +IN at GND (previously
  U13-D was left floating).
- Passive references, values and symbol UUIDs are unchanged, so the PCB
  footprints stay linked.

3. SENSORS sheet readability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
Other:
- sheet POWER SUPPLY - ADC - SACRIFIED SENSOR ports: added Vsac; removed none
- sheet SENSORS ports: added Vsac; removed none
Changed lines of the file:
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@@
+		)
+	)
+	(wire
+		(pts
+			(xy 138.43 90.17) (xy 138.43 115.57)
+		)
+		(stroke
+			(width 0)
+			(type default)
+		)
+	)
+	(wire
+		(pts
+			(xy 35.56 115.57) (xy 35.56 97.79)
+		)
+		(stroke
+			(width 0)
+			(type default)
+		)
+	)
+	(wire
+		(pts
+			(xy 138.43 115.57) (xy 35.56 115.57)
+		)
+		(stroke
+			(width 0)
+			(type default)
+		)
+	)
+	(wire
+		(pts
+			(xy 151.13 90.17) (xy 138.43 90.17)
+		)
+		(stroke
+			(width 0)
+			(type default)
+		)
+	)
+	(wire
+		(pts
+			(xy 35.56 97.79) (xy 40.64 97.79)
+		)
+		(stroke
+			(width 0)
+			(type default)
 		)
 	)
@@
 			)
 		)
+		(pin "Vsac" output
+			(at 151.13 90.17 180)
+			(effects
+				(font
+					(size 1.27 1.27)
+				)
+				(justify left)
+			)
+		)
 		(pin "Vout4" input
 			(at 151.13 80.01 180)
@@
 			(effects
 				(font
+					(size 1.27 1.27)
+				)
+				(justify left)
+			)
+		)
+		(pin "Vsac" input
+			(at 40.64 97.79 180)
+			(effects
+				(font
