File: PCB/FOGLIO1.kicad_sch (KiCad schematic)
At the start: 35 parts, among them J1 Conn_01x02_Pin, J3 6871XX182122_687110182122, J5 Conn_01x03_Pin, J7 Conn_01x07_Pin, U1 LT3483AxS6, U2 LT1761-2.5, U3 LT1964-BYP, U5 AD7606

Commit message: Modifiche accordate fatte
Other:
- moved on the sheet: L1

Commit message: Added decoupling on LDOs, continued optimized power layout, changed packages of 1uF caps
Parts:
- added C48, C49: 1u, Capacitor_SMD:C_0603_1608Metric, symbol Device:C
- C45: footprint Capacitor_SMD:C_0805_2012Metric -> Capacitor_SMD:C_0603_1608Metric
- C5: symbol Device:C_Polarized_Small_US -> Device:C_Small
Connections:
- net +5V: now also C49.1
- net -5V: now also C48.1
- net GND: now also C48.2, C49.2

Commit message: Changed power, started changing ADC and refactoring signal amplitude
Parts:
- removed C1: 4.7u, Capacitor_SMD:C_0805_2012Metric, symbol Device:C
- removed C2: 22p, Capacitor_SMD:C_0603_1608Metric, symbol Device:C
- removed C3, C42: 10u, Capacitor_SMD:C_0805_2012Metric, symbol Device:C
- removed C4: 10u, Capacitor_SMD:C_0805_2012Metric, symbol Device:C_Polarized_Small_US
- removed C48, C49: 1u, Capacitor_SMD:C_0603_1608Metric, symbol Device:C
- removed C5: 0.01u, Capacitor_SMD:C_0603_1608Metric, symbol Device:C_Small
- removed D1: BAT760-7, BAT760-7 diodo:SOD2513X120N, symbol BAT760-7:BAT760-7
- removed J1: Conn_01x02_Pin, Connector_PinHeader_2.54mm:PinHeader_1x02_P2.54mm_Vertical_SMD_Pin1Right, symbol Connector:Conn_01x02_Pin
- removed L1: SDQ12-4R7-R, COILTRONICS SDQ12-4R7 INDUTTORI ACCOPPIATI:INDM5252X12N, symbol SDQ12-4R7-R:SDQ12-4R7-R
- removed R3: 511k, Resistor_SMD:R_0603_1608Metric, symbol Device:R
- removed R4: 105k, Resistor_SMD:R_0603_1608Metric, symbol Device:R
- removed R5: 100k, Resistor_SMD:R_0603_1608Metric, symbol Device:R
- removed TP4: TestPoint, TestPoint:TestPoint_Pad_D1.5mm, symbol Connector:TestPoint
- removed U1: LT3483AxS6, Package_TO_SOT_SMD:TSOT-23-6, symbol Regulator_Switching:LT3483AxS6
- removed U2: LT1761-2.5, Package_TO_SOT_SMD:TSOT-23-5, symbol Regulator_Linear:LT1761-2.5
- removed U3: LT1964-BYP, Package_TO_SOT_SMD:TSOT-23-5, symbol Regulator_Linear:LT1964-BYP
- added C17, C21, C34: 10u, Capacitor_SMD:C_0805_2012Metric, symbol Device:C
- added C19, C20: 4.7u, Capacitor_SMD:C_0603_1608Metric, symbol Device:C_Small
- added C29, C30, C31, C32, C7, C9: 100n, Capacitor_SMD:C_0603_1608Metric, symbol Device:C_Small
- added C33: 100n, Capacitor_SMD:C_0603_1608Metric, symbol Device:C
- added C35: 220n, Capacitor_SMD:C_0603_1608Metric, symbol Device:C_Small
- added C36, C37, C6: 1u, Capacitor_SMD:C_0603_1608Metric, symbol Device:C_Small
- added J2: USB_C_Receptacle_PowerOnly_6P, Connector_USB:USB_C_Receptacle_GCT_USB4125-xx-x_6P_TopMnt_Horizontal, symbol Connector:USB_C_Receptacle_PowerOnly_6P
- added R1: 130k, PCM_SparkFun-Resistor:R_0603_1608Metric, symbol Device:R_Small
- added R11, R12: 10k, PCM_SparkFun-Resistor:R_0603_1608Metric, symbol Device:R_Small
- added R2: 105k, PCM_SparkFun-Resistor:R_0603_1608Metric, symbol Device:R_Small
- added R3, R4: 5.1k, PCM_SparkFun-Resistor:R_0603_1608Metric, symbol Device:R_Small
- added R6: 120k, PCM_SparkFun-Resistor:R_0603_1608Metric, symbol Device:R_Small
- added R9: 100k, PCM_SparkFun-Resistor:R_0603_1608Metric, symbol Device:R_Small
- added U1: TPD2E2U06DCK, Package_TO_SOT_SMD:SOT-323_SC-70, symbol Power_Protection:TPD2E2U06DCK
- added U2: ADS131M08xPBS, Package_QFP:TQFP-32_5x5mm_P0.5mm, symbol Analog_ADC:ADS131M08xPBS
- added U3: 74LVC1G17, symbol 74xGxx:74LVC1G17
- added U4: LM27762, Package_SON:WSON-12-1EP_3x2mm_P0.5mm_EP1x2.65_ThermalVias, symbol Regulator_SwitchedCapacitor:LM27762
Connections:
- net +2V5: now also C20.1, C9.1, R1.1, U4.11 (OUT+)
- net +5V: now also C21.1, C29.2, C30.2, C31.2, C33.1, C34.1, J2.A9 (VBUS), J2.B9 (VBUS), R11.1, R12.1, U4.3 (VIN)
- net -2V5: now also C19.2, C7.2, R2.2, U4.6 (OUT-)
- net GND: now also C17.2, C19.1, C20.2, C21.2, C29.1, C30.1, C31.1, C32.1, C33.2, C34.2, C35.2, C36.2, C37.2, C7.1, C9.2, J2.A12 (GND), J2.B12 (GND), J2.SH (SHIELD), R3.2, R4.2, R6.2, R9.2, U1.3, U2.10 (AIN6N), U2.11 (AIN7N), U2.13 (AGND), U2.2 (AIN2N), U2.25 (DGND), U2.27 (AGND), U2.28 (AGND), U2.3 (AIN3N), U2.30 (AIN0N), U2.31 (AIN1N), U2.6 (AIN4N), U2.7 (AIN5N), U3.3 (GND), U4.13 (PAD), U4.4 (GND); no longer U5.50 (V1GND), U5.52 (V2GND), U5.54 (V3GND), U5.56 (V4GND), U5.58 (V5GND), U5.60 (V6GND), U5.62 (V7GND)
- net Vdrive: now also C32.2
- net Vout1: now also U2.29 (AIN0P); no longer U5.49 (V1)
- net Vout2: now also U2.32 (AIN1P); no longer U5.51 (V2)
- net Vout3: now also U2.1 (AIN2P); no longer U5.53 (V3)
- net Vout4: now also U2.4 (AIN3P); no longer U5.55 (V4)
- net Vout5: now also U2.5 (AIN4P); no longer U5.57 (V5)
- net Vout6: now also U2.8 (AIN5P); no longer U5.59 (V6)
- net Vout7: now also U2.9 (AIN6P); no longer U5.61 (V7)
- new net: C37.1, U2.15 (AVDD)
- new net: U2.23 (XTAL1/CLKIN), U3.4
- new net: C35.1, U2.24 (CAP)
- new net: C36.1, U2.26 (DVDD)
- new net: R2.1, R9.1, U4.7 (FB-)
- new net: R12.2, U4.12 (EN+), U4.8 (EN-)
- new net: C17.1, U4.5 (CP)
- new net: R11.2, U4.1 (PGOOD)
- new net: C6.1, U4.10 (C+)
- new net: R1.2, R6.1, U4.2 (FB+)
- new net: C6.2, U4.9 (C-)
- new net: J2.A5 (CC1), R4.1, U1.1
- new net: J2.B5 (CC2), R3.1, U1.2
- new net +3V3: U3.5 (VCC)
- new net MCU_CLK: U3.2
- new net Vsac: U2.12 (AIN7P)
Other:
- note added: "MOUNTING HOLES"
- note added: "POWER STAGE: INTEGRATED CHARGE PUMP INVERTER + LDOs 5V-> +/- 2V5"
- note added: "POWER SUPPLY (USBC)"
- note removed: "Converting 5V to -5V"
- note removed: "DC-DC: 5V DOWN TO -5V"
- note removed: "MOUNTIG HOLES"
- note removed: "POWER SUPPLY"
- note removed: "REGULATOR: -5V UP TO -2.5V"
- note removed: "REGULATOR: 5V DOWN TO 2.5V"
- moved on the sheet: TP1, TP2, TP3
